File: controller/hardware_design/pcb/max/Mobo-v09.sch (EAGLE design)
At the start: 137 parts, among them IC1 TL072, IC10 74HC595N, IC11 74HC595N, IC2 MCP1700, IC3 4050N, IC4 74HC138N, IC5 7908, IC6 2940T-8.0, IC7 7805, IC8 ATMEGA644p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

Commit message: refactoring of variable names and computations, still can't find the final bug...
Other:
- note added: "Emilie Gillet, 2011. cc-by-sa"
- note removed: "Olivier Gillet, 2011. cc-by-sa"
Changed lines of the file:
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@@
 <plain>
 <text x="45.72" y="-73.66" size="3.81" layer="94" ratio="15">Main MCU / digital plumbing</text>
-<text x="45.72" y="-78.74" size="2.54" layer="94">Olivier Gillet, 2011. cc-by-sa</text>
+<text x="45.72" y="-78.74" size="2.54" layer="94">Emilie Gillet, 2011. cc-by-sa</text>
 </plain>
 <instances>
@@
 <text x="25.4" y="-15.24" size="3.81" layer="94" ratio="15">User interface</text>
 <text x="93.98" y="124.46" size="1.778" layer="97">Duo-color LEDs</text>
-<text x="25.4" y="-20.32" size="2.54" layer="94">Olivier Gillet, 2011. cc-by-sa</text>
+<text x="25.4" y="-20.32" size="2.54" layer="94">Emilie Gillet, 2011. cc-by-sa</text>
 </plain>
 <instances>
@@
 <plain>
 <text x="33.02" y="88.9" size="3.81" layer="94" ratio="15">Peripherals</text>
-<text x="33.02" y="83.82" size="2.54" layer="94">Olivier Gillet, 2011. cc-by-sa</text>
+<text x="33.02" y="83.82" size="2.54" layer="94">Emilie Gillet, 2011. cc-by-sa</text>
 <text x="-93.98" y="198.12" size="1.9304" layer="97" ratio="15" rot="R90">Port 7</text>
 </plain>
@@
 <plain>
 <text x="40.64" y="-48.26" size="3.81" layer="94" ratio="15">Voicecards and mixing</text>
-<text x="40.64" y="-53.34" size="2.54" layer="94">Olivier Gillet, 2011. cc-by-sa</text>
+<text x="40.64" y="-53.34" size="2.54" layer="94">Emilie Gillet, 2011. cc-by-sa</text>
 <text x="15.24" y="106.68" size="1.9304" layer="97" ratio="15" rot="R270">Port 1-2</text>
 <text x="15.24" y="60.96" size="1.9304" layer="97" ratio="15" rot="R270">Port 3-4</text>
@@
 <text x="-7.62" y="76.2" size="1.778" layer="97">9V AC, 1A</text>
 <text x="83.82" y="-2.54" size="3.81" layer="94" ratio="15">Power supply</text>
-<text x="83.82" y="-7.62" size="2.54" layer="94">Olivier Gillet, 2011. cc-by-sa</text>
+<text x="83.82" y="-7.62" size="2.54" layer="94">Emilie Gillet, 2011. cc-by-sa</text>
 <text x="88.9" y="93.98" size="1.778" layer="97">130mA</text>
 <text x="88.9" y="50.8" size="1.778" layer="97">130mA</text>
